Commit message: Unify robot description and lidar TF ownership

File: src/turn_on_wheeltec_robot/urdf/patrol_robot.urdf.xacro (robot description, xacro)
@@ -1,12 +1,19 @@
 <?xml version="1.0"?>
 <robot xmlns:xacro="http://www.ros.org/wiki/xacro" name="patrol_robot_vertical">
-  <xacro:property name="base_length" value="0.400" />
-  <xacro:property name="base_width"  value="0.350" />
-  <xacro:property name="base_box_height" value="0.745" />
-  <xacro:property name="base_ground_clearance" value="0.0785" />
-  <xacro:property name="lidar_offset_x" value="0.190" />
-  <xacro:property name="lidar_offset_y" value="0.000" />
-  <xacro:property name="lidar_offset_z" value="0.550" />
-  <xacro:property name="lidar_rpy" value="0.0 1.5708 0.0" />
+  <xacro:property name="base_length" value="0.400"/>
+  <xacro:property name="base_width" value="0.350"/>
+  <xacro:property name="base_box_height" value="0.745"/>
+  <xacro:property name="base_ground_clearance" value="0.0785"/>
+  <xacro:property name="lidar_offset_x" value="0.190"/>
+  <xacro:property name="lidar_offset_y" value="0.000"/>
+  <xacro:property name="lidar_offset_z" value="0.550"/>
+  <!-- Mechanical mounting frame fixed to the chassis. -->
+  <xacro:property name="lidar_mount_rpy" value="0.0 1.5708 3.14159"/>
+  <!-- Verified Unitree driver-frame correction: roll=pi, yaw=115.234 deg. -->
+  <xacro:property name="lidar_driver_rpy" value="3.14159 0.0 2.0112063268"/>
+  <!-- Unitree factory IMU origin expressed in the LiDAR frame. Axes are parallel. -->
+  <xacro:property name="imu_offset_x" value="-0.007698"/>
+  <xacro:property name="imu_offset_y" value="-0.014655"/>
+  <xacro:property name="imu_offset_z" value="0.00667"/>
   <link name="base_footprint"/>
   <joint name="base_joint" type="fixed">
@@ -35,5 +42,23 @@
     <parent link="base_link"/>
     <child link="unilidar_link"/>
-    <origin xyz="${lidar_offset_x} ${lidar_offset_y} ${lidar_offset_z}" rpy="${lidar_rpy}"/>
+    <origin
+      xyz="${lidar_offset_x} ${lidar_offset_y} ${lidar_offset_z}"
+      rpy="${lidar_mount_rpy}"/>
+  </joint>
+  <!-- Driver-published PointCloud2 frame. This is the single TF authority. -->
+  <link name="unilidar_lidar"/>
+  <joint name="unilidar_lidar_joint" type="fixed">
+    <parent link="unilidar_link"/>
+    <child link="unilidar_lidar"/>
+    <origin xyz="0 0 0" rpy="${lidar_driver_rpy}"/>
+  </joint>
+  <!-- Driver-published IMU frame, parallel to the LiDAR axes per Unitree. -->
+  <link name="unilidar_imu"/>
+  <joint name="unilidar_imu_joint" type="fixed">
+    <parent link="unilidar_lidar"/>
+    <child link="unilidar_imu"/>
+    <origin
+      xyz="${imu_offset_x} ${imu_offset_y} ${imu_offset_z}"
+      rpy="0 0 0"/>
   </joint>
 </robot>

Commit message: Use measured chassis envelope for Nav2

File: src/turn_on_wheeltec_robot/urdf/patrol_robot.urdf.xacro (robot description, xacro)
@@ -1,6 +1,7 @@
 <?xml version="1.0"?>
 <robot xmlns:xacro="http://www.ros.org/wiki/xacro" name="patrol_robot_vertical">
-  <xacro:property name="base_length" value="0.400"/>
-  <xacro:property name="base_width" value="0.350"/>
+  <!-- Conservative measured outer envelope, including protruding hardware. -->
+  <xacro:property name="base_length" value="0.510"/>
+  <xacro:property name="base_width" value="0.410"/>
   <xacro:property name="base_box_height" value="0.745"/>
   <xacro:property name="base_ground_clearance" value="0.0785"/>

Commit message: fix nav mode recovery and rotate lidar mount

File: src/turn_on_wheeltec_robot/urdf/patrol_robot.urdf.xacro (robot description, xacro)
@@ -9,6 +9,7 @@
   <xacro:property name="lidar_offset_y" value="0.000"/>
   <xacro:property name="lidar_offset_z" value="0.550"/>
-  <!-- Mechanical mounting frame fixed to the chassis. -->
-  <xacro:property name="lidar_mount_rpy" value="0.0 1.5708 3.14159"/>
+  <!-- Mechanical mounting frame fixed to the chassis. The chassis-facing yaw
+       is 90 deg clockwise from the previous pi-radian assumption. -->
+  <xacro:property name="lidar_mount_rpy" value="0.0 1.5708 1.5707963268"/>
   <!-- Verified Unitree driver-frame correction: roll=pi, yaw=115.234 deg. -->
   <xacro:property name="lidar_driver_rpy" value="3.14159 0.0 2.0112063268"/>

Commit message: add visual lidar yaw calibration

File: src/turn_on_wheeltec_robot/urdf/patrol_robot.urdf.xacro (robot description, xacro)
@@ -1,4 +1,5 @@
 <?xml version="1.0"?>
 <robot xmlns:xacro="http://www.ros.org/wiki/xacro" name="patrol_robot_vertical">
+  <xacro:arg name="lidar_mount_yaw_rad" default="3.14159"/>
   <!-- Conservative measured outer envelope, including protruding hardware. -->
   <xacro:property name="base_length" value="0.510"/>
@@ -9,7 +10,7 @@
   <xacro:property name="lidar_offset_y" value="0.000"/>
   <xacro:property name="lidar_offset_z" value="0.550"/>
-  <!-- Mechanical mounting frame fixed to the chassis. The chassis-facing yaw
-       is 90 deg clockwise from the previous pi-radian assumption. -->
-  <xacro:property name="lidar_mount_rpy" value="0.0 1.5708 1.5707963268"/>
+  <!-- Mechanical mounting frame fixed to the chassis. The yaw is operator
+       calibrated from the Ubuntu console and stored in the Orin allowlist. -->
+  <xacro:property name="lidar_mount_rpy" value="0.0 1.5708 $(arg lidar_mount_yaw_rad)"/>
   <!-- Verified Unitree driver-frame correction: roll=pi, yaw=115.234 deg. -->
   <xacro:property name="lidar_driver_rpy" value="3.14159 0.0 2.0112063268"/>

Commit message: upgrade lidar calibration to three-axis RViz preview

File: src/turn_on_wheeltec_robot/urdf/patrol_robot.urdf.xacro (robot description, xacro)
@@ -1,4 +1,6 @@
 <?xml version="1.0"?>
 <robot xmlns:xacro="http://www.ros.org/wiki/xacro" name="patrol_robot_vertical">
+  <xacro:arg name="lidar_mount_roll_rad" default="0.0"/>
+  <xacro:arg name="lidar_mount_pitch_rad" default="1.5708"/>
   <xacro:arg name="lidar_mount_yaw_rad" default="3.14159"/>
   <!-- Conservative measured outer envelope, including protruding hardware. -->
@@ -12,5 +14,5 @@
   <!-- Mechanical mounting frame fixed to the chassis. The yaw is operator
        calibrated from the Ubuntu console and stored in the Orin allowlist. -->
-  <xacro:property name="lidar_mount_rpy" value="0.0 1.5708 $(arg lidar_mount_yaw_rad)"/>
+  <xacro:property name="lidar_mount_rpy" value="$(arg lidar_mount_roll_rad) $(arg lidar_mount_pitch_rad) $(arg lidar_mount_yaw_rad)"/>
   <!-- Verified Unitree driver-frame correction: roll=pi, yaw=115.234 deg. -->
   <xacro:property name="lidar_driver_rpy" value="3.14159 0.0 2.0112063268"/>
